Commit message: feat(description): mount Ouster OS-1 on the bottom shelf board (relocated + yaw-flipped)
Move the OS-1 from shelf_top to shelf_bottom_board (os_lidar ~0.65 -> ~0.166 m
above base_link) and yaw-flip the shelf+sensor assembly 180 deg about Z to match
the physical mounting (RViz-verified on hardware). Add the description package's
first pytest (xacro-expansion check of the mount height + parent).

Signed-off-by: Yutaka Kondo <yutaka.kondo@youtalk.jp>

File: kachaka_autoware_description/urdf/kachaka_with_shelf.urdf.xacro (robot description, xacro)
@@ -18,13 +18,21 @@
     (up to +0.012 m) because docking_link is a prismatic child of base_link.
   -->
+  <!-- Yaw 180 deg (rpy 0 0 PI): the shelf + OS-1 assembly is physically mounted
+       facing the robot's rear, so flip it about Z to match reality (RViz-verified
+       2026-07-10). This rotates the mounted Ouster's extrinsic too, so the cloud
+       aligns with base_link. -->
   <xacro:shelf_3tier parent="docking_link">
-    <origin xyz="0 0 0.115" rpy="0 0 0"/>
+    <origin xyz="0 0 0.115" rpy="0 0 ${PI}"/>
   </xacro:shelf_3tier>
-  <!-- Mount the Ouster OS-1 at the shelf top center; override origin with values measured in M0 Task 4.
-       name="os" so URDF link names (os_sensor / os_lidar / os_imu) match the ouster_ros driver's default
-       sensor_frame / lidar_frame / imu_frame; otherwise the published cloud's frame_id is unconnected
-       to the robot TF tree and downstream NDT / snapshot tools fail to look up the transform. -->
-  <xacro:ouster_os1 parent="shelf_top" name="os">
-    <origin xyz="0 0 0" rpy="0 0 0"/>
+  <!-- Mount the Ouster OS-1 on the bottom shelf board (relocated 2026-07 from
+       shelf_top to lower the sensor to ~0.17 m above base_link, enabling ground-filter
+       experiments). shelf_bottom_board's link frame sits at the shelf base; origin z is
+       one board thickness (0.015) so the sensor body rests on the board's top surface.
+       Override origin with the M0-measured mount pose. name="os" so URDF link names
+       (os_sensor / os_lidar / os_imu) match the ouster_ros driver's default sensor_frame /
+       lidar_frame / imu_frame; otherwise the published cloud's frame_id is unconnected to
+       the robot TF tree and downstream NDT / snapshot tools fail to look up the transform. -->
+  <xacro:ouster_os1 parent="shelf_bottom_board" name="os">
+    <origin xyz="0 0 0.015" rpy="0 0 0"/>
   </xacro:ouster_os1>
 </robot>

Commit message: feat: 3D LiDAR bottom-shelf relocation + OS-1 TF for NDT (#16)
* feat(description): mount Ouster OS-1 on the bottom shelf board (relocated + yaw-flipped)

Move the OS-1 from shelf_top to shelf_bottom_board (os_lidar ~0.65 -> ~0.166 m
above base_link) and yaw-flip the shelf+sensor assembly 180 deg about Z to match
the physical mounting (RViz-verified on hardware). Add the description package's
first pytest (xacro-expansion check of the mount height + parent).

Signed-off-by: Yutaka Kondo <yutaka.kondo@youtalk.jp>

* feat(bridge): publish shelf+OS-1 TF in LiDAR modes so NDT gets the OS-1 cloud

In the loc_lidar group of kachaka_autoware_2d.launch.xml, start the shelf+OS-1
robot_state_publisher so base_link -> os_lidar TF exists for NDT (shadow/ndt).
The body RSP from _grpc_bridge_core still owns the body/base_link edges; the
superset URDF re-publishes those identical static edges (benign).

Signed-off-by: Yutaka Kondo <yutaka.kondo@youtalk.jp>

* feat: add with_shelf toggle (shelf+OS-1 vs bare Kachaka body)

with_shelf xacro arg (default true) wraps the shelf_3tier + OS-1 in the URDF;
robot_description.launch.py forwards it to xacro. In kachaka_autoware_2d.launch.xml
a with_shelf launch arg gates a run_shelf group that publishes the shelf+OS-1
robot_state_publisher; it is forced on in shadow/ndt (the OS-1 rides the shelf and
NDT needs base_link->os_lidar). with_shelf:=false brings up the bare body.
Extend test_urdf_mount with a with_shelf:=false bare-body case.

Signed-off-by: Yutaka Kondo <yutaka.kondo@youtalk.jp>

* chore: remove superseded kachaka_autoware.launch.xml (PR review)

Delete the legacy all-in-one entry point kachaka_autoware.launch.xml (replaced by
the verified kachaka_autoware_2d.launch.xml) and its only consumer
launch/localization.launch.xml (orphaned by the deletion). Point the
kachaka_autoware_maps README at the 2D entry point (localization_mode:=ndt).
Addresses PR review: '必要なくなったなら削除する'.

Signed-off-by: Yutaka Kondo <yutaka.kondo@youtalk.jp>

* fix(description): vendor _shelf_3tier.urdf.xacro so the shelf URDF expands in CI

CI's colcon test failed on test_urdf_mount: 'xacro ... No such file or directory
.../kachaka_description/.../_shelf_3tier.urdf.xacro' (exit 2). The 3-tier shelf
macro is a local addition the upstream kachaka-api submodule does not ship, so a
clean checkout could not resolve $(find kachaka_description)/urdf/_shelf_3tier.
Vendor it into kachaka_autoware_description (which models the Autoware shelf) and
include it from there. _materials/_values/_kachaka still come from the submodule,
which does track them. Verified: colcon test kachaka_autoware_description -> 3/3.

Signed-off-by: Yutaka Kondo <yutaka.kondo@youtalk.jp>

* fix(bridge): publish shelf+OS-1 RSP at root to avoid /kachaka RSP node collision

Hardware final check found the shelf+OS-1 robot_state_publisher (run_shelf group)
running as /kachaka/robot_state_publisher, colliding with the body RSP from
_grpc_bridge_core on both the node name AND the /kachaka/robot_description topic.
The collision corrupts the TF tree: base_link->os_lidar was non-deterministic,
flipping between yaw 0 and yaw 180 across launches/lookups. Publish the shelf RSP
at the root namespace (namespace="") -> /robot_state_publisher +
/robot_description, distinct from the body's. frame_prefix stays empty so frame
ids remain global. Verified on hardware: base_link->os_lidar = yaw 180 stable
across 3 lookups, cloud 10 Hz, RobotModel + TF render cleanly.

Signed-off-by: Yutaka Kondo <yutaka.kondo@youtalk.jp>

* refactor(launch): rename kachaka_autoware_2d.launch.xml to kachaka_autoware.launch.xml

PR #16 removed the original kachaka_autoware.launch.xml, leaving the _2d
variant as the sole entry point. Since _2d now covers both the 2D Kachaka
SLAM passthrough and the 3D-LiDAR NDT/shadow modes via localization_mode,
the suffix no longer distinguishes anything. Rename it back to the plain
name and update every in-repo reference (endurance/canned_trajectory
launches, both package READMEs, stitch_map launch + script).

The rviz/kachaka_autoware_2d.rviz config keeps its name (separate artifact).

Signed-off-by: Yutaka Kondo <yutaka.kondo@youtalk.jp>

* refactor(rviz): drop _2d suffix from rviz config to match launch rename

Complete the _2d suffix removal: rename kachaka_autoware_2d.rviz to
kachaka_autoware.rviz and repoint the launch rviz_config default. Now no
kachaka_autoware_2d name remains in the package. (The _2d tokens left in
the vendored kachaka-api submodule are upstream ROS names — nav2_costmap_2d,
calculate_2d_transform_matrix — not our suffix.)

Signed-off-by: Yutaka Kondo <yutaka.kondo@youtalk.jp>

---------

Signed-off-by: Yutaka Kondo <yutaka.kondo@youtalk.jp>

File: kachaka_autoware_description/urdf/kachaka_with_shelf.urdf.xacro (robot description, xacro)
@@ -4,10 +4,14 @@
   <xacro:include filename="$(find kachaka_description)/urdf/_values.urdf.xacro"/>
   <xacro:include filename="$(find kachaka_description)/urdf/_kachaka.urdf.xacro"/>
-  <xacro:include filename="$(find kachaka_description)/urdf/_shelf_3tier.urdf.xacro"/>
+  <xacro:include filename="$(find kachaka_autoware_description)/urdf/_shelf_3tier.urdf.xacro"/>
   <xacro:include filename="$(find kachaka_autoware_description)/urdf/_ouster_os1.urdf.xacro"/>
+  <!-- with_shelf:=false publishes the bare Kachaka body only (no 3-tier shelf,
+       no OS-1). Default true: the robot physically carries the Autoware shelf. -->
+  <xacro:arg name="with_shelf" default="true"/>
   <link name="base_footprint"/>
   <xacro:kachaka_robot parent="base_footprint">
     <origin xyz="0 0 0" rpy="0 0 0"/>
   </xacro:kachaka_robot>
+  <xacro:if value="$(arg with_shelf)">
   <!--
     docking_link is Kachaka's docking lift mechanism (prismatic joint).
@@ -18,13 +22,22 @@
     (up to +0.012 m) because docking_link is a prismatic child of base_link.
   -->
+  <!-- Yaw 180 deg (rpy 0 0 PI): the shelf + OS-1 assembly is physically mounted
+       facing the robot's rear, so flip it about Z to match reality (RViz-verified
+       2026-07-10). This rotates the mounted Ouster's extrinsic too, so the cloud
+       aligns with base_link. -->
   <xacro:shelf_3tier parent="docking_link">
-    <origin xyz="0 0 0.115" rpy="0 0 0"/>
+    <origin xyz="0 0 0.115" rpy="0 0 ${PI}"/>
   </xacro:shelf_3tier>
-  <!-- Mount the Ouster OS-1 at the shelf top center; override origin with values measured in M0 Task 4.
-       name="os" so URDF link names (os_sensor / os_lidar / os_imu) match the ouster_ros driver's default
-       sensor_frame / lidar_frame / imu_frame; otherwise the published cloud's frame_id is unconnected
-       to the robot TF tree and downstream NDT / snapshot tools fail to look up the transform. -->
-  <xacro:ouster_os1 parent="shelf_top" name="os">
-    <origin xyz="0 0 0" rpy="0 0 0"/>
+  <!-- Mount the Ouster OS-1 on the bottom shelf board (relocated 2026-07 from
+       shelf_top to lower the sensor to ~0.17 m above base_link, enabling ground-filter
+       experiments). shelf_bottom_board's link frame sits at the shelf base; origin z is
+       one board thickness (0.015) so the sensor body rests on the board's top surface.
+       Override origin with the M0-measured mount pose. name="os" so URDF link names
+       (os_sensor / os_lidar / os_imu) match the ouster_ros driver's default sensor_frame /
+       lidar_frame / imu_frame; otherwise the published cloud's frame_id is unconnected to
+       the robot TF tree and downstream NDT / snapshot tools fail to look up the transform. -->
+  <xacro:ouster_os1 parent="shelf_bottom_board" name="os">
+    <origin xyz="0 0 0.015" rpy="0 0 0"/>
   </xacro:ouster_os1>
+  </xacro:if>
 </robot>
