Commit message: fix(description): encode the OS-1 lidar->sensor 180 deg yaw on the lidar joint
The point cloud is expressed in os_lidar, which per the Ouster ICD
(metadata lidar_to_sensor_transform = diag(-1,-1,1) + z) is yawed 180 deg
about Z from os_sensor. The URDF os_sensor->os_lidar joint had rpy 0 0 0,
so it disagreed with the static TF the driver publishes itself
(pub_static_tf:=true, the correct 180 deg). The two static publishers
raced, so base_link->os_lidar flipped nondeterministically between 0 and
180 deg and the cloud rendered 180 deg off.

Encode the ICD yaw on the os_sensor->os_lidar joint (rpy 0 0 PI) so the
URDF matches the driver and the transform is deterministic. Drop the
compensating 180 deg yaw that was on the shelf mount: the shelf/OS-1
assembly faces forward (the "rear-facing" note was a mis-diagnosis made
while the cloud was mis-timestamped and never rendered in map). Net
base_link->os_lidar is unchanged (180 deg yaw, z 0.16618) but os_sensor /
os_imu now face the right way and the result no longer races.

test_urdf_mount still passes (height/parent unaffected; the only rotation
on the chain is still a Z yaw); its note is updated to point at the joint
that now carries the yaw.

Signed-off-by: Yutaka Kondo <yutaka.kondo@youtalk.jp>

File: kachaka_autoware_description/urdf/_ouster_os1.urdf.xacro (robot description, xacro)
@@ -37,9 +37,14 @@
       <xacro:insert_block name="origin"/>
     </joint>
+    <!-- os_lidar is yawed 180 deg about Z relative to os_sensor per the Ouster ICD
+         (metadata lidar_to_sensor_transform = diag(-1,-1,1) + z). The point cloud data
+         is expressed in os_lidar, and the driver publishes this same static TF
+         (pub_static_tf:=true); this joint MUST match it (rpy 0 0 PI) or the two
+         os_sensor->os_lidar publishers disagree and the cloud renders 180 deg flipped. -->
     <link name="${name}_lidar"/>
     <joint name="${name}_lidar_joint" type="fixed">
       <parent link="${name}_sensor"/>
       <child link="${name}_lidar"/>
-      <origin xyz="0 0 ${lidar_to_sensor_z}" rpy="0 0 0"/>
+      <origin xyz="0 0 ${lidar_to_sensor_z}" rpy="0 0 ${PI}"/>
     </joint>
     <link name="${name}_imu"/>

File: kachaka_autoware_description/urdf/kachaka_with_shelf.urdf.xacro (robot description, xacro)
@@ -22,10 +22,11 @@
     (up to +0.012 m) because docking_link is a prismatic child of base_link.
   -->
-  <!-- Yaw 180 deg (rpy 0 0 PI): the shelf + OS-1 assembly is physically mounted
-       facing the robot's rear, so flip it about Z to match reality (RViz-verified
-       2026-07-10). This rotates the mounted Ouster's extrinsic too, so the cloud
-       aligns with base_link. -->
+  <!-- No yaw: the shelf + OS-1 assembly is mounted facing forward, aligned with
+       base_link. (An earlier rpy="0 0 PI" yaw flip was a mis-diagnosis made while
+       the OS-1 cloud was mis-timestamped and not rendering in the map frame; with
+       the cloud correctly displayed it is 180 deg off, so the flip is removed —
+       RViz-verified 2026-07-10.) -->
   <xacro:shelf_3tier parent="docking_link">
-    <origin xyz="0 0 0.115" rpy="0 0 ${PI}"/>
+    <origin xyz="0 0 0.115" rpy="0 0 0"/>
   </xacro:shelf_3tier>
   <!-- Mount the Ouster OS-1 on the bottom shelf board (relocated 2026-07 from
